Commit message: urdf working with texture

File: simulation/urdf/rover.urdf (robot description, URDF)
Before this commit: robot rover, 14 links, 13 joints
Links:
- link Wheel_Link_BL: geometry collision mesh filename=package://rover/meshes/Wheel_Link_BL.STL; visual mesh filename=package://rover/textures/Wheel_Link_BL.dae
